Commit message: controller

File: urdf/squid.urdf (robot description, URDF)
Before this commit: robot three_arm_octobot, 125 links, 124 joints
Links:
- added link imu_link, mass 0.01; collision box size=0.03 0.03 0.01; visual box size=0.03 0.03 0.01
Joints:
- added joint head_to_imu: type fixed, parent head, child imu_link, origin xyz=0 0 0.05 rpy=0 0 0
